Commit message: some other issue with the new model

File: bandu_stacking/models/srl/franka_research_panda/panda.urdf (robot description, URDF)
Before this commit: robot fr3, 14 links, 13 joints
Links:
- removed link fr3_hand
- removed link fr3_hand_tcp
- removed link fr3_leftfinger
- removed link fr3_link0
- removed link fr3_link1
- removed link fr3_link2
- removed link fr3_link3
- removed link fr3_link4
- removed link fr3_link5
- removed link fr3_link6
- removed link fr3_link7
- removed link fr3_link8
- removed link fr3_rightfinger
- added link panda_hand, mass 0.73; collision mesh filename=package://meshes/fr3/collision/hand.stl; visual mesh filename=package://meshes/fr3/visual/hand.dae
- added link panda_hand_tcp
- added link panda_leftfinger; collision box size=17.5e-3 15.2e-3 18.5e-3; collision box size=17.5e-3 7e-3 23.5e-3
- added link panda_link0; collision mesh filename=package://meshes/fr3/collision/link0.stl; visual mesh filename=package://meshes/fr3/visual/link0.dae
- added link panda_link1, mass 2.9274653454; collision mesh filename=package://meshes/fr3/collision/link1.stl; visual mesh filename=package://meshes/fr3/visual/link1.dae
- added link panda_link2, mass 2.9355370338; collision mesh filename=package://meshes/fr3/collision/link2.stl; visual mesh filename=package://meshes/fr3/visual/link2.dae
- added link panda_link3, mass 2.2449013699; collision mesh filename=package://meshes/fr3/collision/link3.stl; visual mesh filename=package://meshes/fr3/visual/link3.dae
- added link panda_link4, mass 2.6155955791; collision mesh filename=package://meshes/fr3/collision/link4.stl; visual mesh filename=package://meshes/fr3/visual/link4.dae
- added link panda_link5, mass 2.3271207594; collision mesh filename=package://meshes/fr3/collision/link5.stl; visual mesh filename=package://meshes/fr3/visual/link5.dae
- added link panda_link6, mass 1.8170376524; collision mesh filename=package://meshes/fr3/collision/link6.stl; visual mesh filename=package://meshes/fr3/visual/link6.dae
- added link panda_link7, mass 0.6271432862; collision mesh filename=package://meshes/fr3/collision/link7.stl; visual mesh filename=package://meshes/fr3/visual/link7.dae
- added link panda_link8
- added link panda_rightfinger; collision box size=17.5e-3 15.2e-3 18.5e-3; collision box size=17.5e-3 7e-3 23.5e-3
- added link panda_tool_tip
Joints:
- removed joint fr3_finger_joint1
- removed joint fr3_finger_joint2
- removed joint fr3_hand_joint
- removed joint fr3_hand_tcp_joint
- removed joint fr3_joint1
- removed joint fr3_joint2
- removed joint fr3_joint3
- removed joint fr3_joint4
- removed joint fr3_joint5
- removed joint fr3_joint6
- removed joint fr3_joint7
- removed joint fr3_joint8
- added joint panda_finger_joint1: type prismatic, parent panda_hand, child panda_leftfinger, origin xyz=0 0 0.0584 rpy=0 0 0, axis 0 1 0, limit lower=0.0 upper=0.04 effort=100 velocity=0.2
- added joint panda_finger_joint2: type prismatic, parent panda_hand, child panda_rightfinger, origin xyz=0 0 0.0584 rpy=0 0 0, axis 0 -1 0, limit lower=0.0 upper=0.04 effort=100 velocity=0.2, mimic joint=panda_finger_joint1
- added joint panda_hand_joint: type fixed, parent panda_link8, child panda_hand, origin xyz=0 0 0 rpy=0 0 -0.7853981633974483
- added joint panda_hand_tcp_joint: type fixed, parent panda_hand, child panda_hand_tcp, origin xyz=0 0 0.1034 rpy=0 0 0
- added joint panda_joint1: type revolute, parent panda_link0, child panda_link1, origin xyz=0 0 0.333 rpy=0 0 0, axis 0 0 1, limit lower=-2.7437 upper=2.7437 effort=87.0 velocity=2.62
- added joint panda_joint2: type revolute, parent panda_link1, child panda_link2, origin xyz=0 0 0 rpy=-1.570796326794897 0 0, axis 0 0 1, limit lower=-1.7837 upper=1.7837 effort=87.0 velocity=2.62
- added joint panda_joint3: type revolute, parent panda_link2, child panda_link3, origin xyz=0 -0.316 0 rpy=1.570796326794897 0 0, axis 0 0 1, limit lower=-2.9007 upper=2.9007 effort=87.0 velocity=2.62
- added joint panda_joint4: type revolute, parent panda_link3, child panda_link4, origin xyz=0.0825 0 0 rpy=1.570796326794897 0 0, axis 0 0 1, limit lower=-3.0421 upper=-0.1518 effort=87.0 velocity=2.62
- added joint panda_joint5: type revolute, parent panda_link4, child panda_link5, origin xyz=-0.0825 0.384 0 rpy=-1.570796326794897 0 0, axis 0 0 1, limit lower=-2.8065 upper=2.8065 effort=12.0 velocity=5.26
- added joint panda_joint6: type revolute, parent panda_link5, child panda_link6, origin xyz=0 0 0 rpy=1.570796326794897 0 0, axis 0 0 1, limit lower=0.5445 upper=4.5169 effort=12.0 velocity=4.18
- added joint panda_joint7: type revolute, parent panda_link6, child panda_link7, origin xyz=0.088 0 0 rpy=1.570796326794897 0 0, axis 0 0 1, limit lower=-3.0159 upper=3.0159 effort=12.0 velocity=5.26
- added joint panda_joint8: type fixed, parent panda_link7, child panda_link8, origin xyz=0 0 0.107 rpy=0 0 0
- added joint panda_tool_tip_joint: type fixed, parent panda_hand, child panda_tool_tip, origin xyz=0 0 0.10 rpy=0 -1.5708 0, axis 0 0 0
- joint base: child fr3_link0 -> panda_link0
